Commit message: Renamed chassi to base link

File: urdf/nubot.gazebo.xacro (robot description, xacro)
@@ -44,5 +44,5 @@
         <odom_publish_frequency>30</odom_publish_frequency>
         <frame_id>odom</frame_id>
-        <child_frame_id>chassis</child_frame_id>
+        <child_frame_id>base_link</child_frame_id>
       </plugin>
       <plugin

File: urdf/nubot.urdf.xacro (robot description, xacro)
@@ -1,4 +1,4 @@
 <robot name="nubot" xmlns:xacro="http://www.ros.org/wiki/xacro">
-      <link name="chassis">
+      <link name="base_link">
         <inertial>
           <origin xyz="-0.151427 -0 0.175" rpy="0 -0 0"/>
@@ -130,10 +130,10 @@
       <joint name="lidar_sensor_joint" type="fixed">
         <origin xyz="0 0 0.5" rpy="0 0 0" />
-        <parent link="chassis" />
+        <parent link="base_link" />
         <child link="lidar_link" />
       </joint>
       <joint name="left_wheel_joint" type="continuous">
         <origin xyz="0.554283 0.625029 -0.025" rpy="-1.5707 0 0" />
-        <parent link="chassis" />
+        <parent link="base_link" />
         <child link="left_wheel" />
         <axis xyz="0 0 1" />
@@ -141,10 +141,10 @@
       <joint name="right_wheel_joint" type="continuous">
         <origin xyz="0.554283 -0.625029 -0.025" rpy="-1.5707 0 0" />
-        <parent link="chassis" />
+        <parent link="base_link" />
         <child link="right_wheel" />
         <axis xyz="0 0 1" />
       </joint>
       <joint name="caster_wheel" type="fixed">
-        <parent link="chassis" />
+        <parent link="base_link" />
         <child link="caster" />
       </joint>

Commit message: Updated lidar_link to be called base_laser

File: urdf/nubot.gazebo.xacro (robot description, xacro)
@@ -4,5 +4,5 @@
           <preserveFixedJoint>true</preserveFixedJoint>
         </gazebo>
-        <gazebo reference="lidar_link" >
+        <gazebo reference="base_laser" >
           <sensor name='gpu_lidar' type='gpu_lidar'>
             <topic>lidar</topic>
@@ -31,5 +31,5 @@
             <alwaysOn>1</alwaysOn>
             <visualize>true</visualize>
-            <ignition_frame_id>lidar_link</ignition_frame_id>
+            <ignition_frame_id>base_laser</ignition_frame_id>
         </sensor>
     </gazebo>

File: urdf/nubot.urdf.xacro (robot description, xacro)
@@ -29,5 +29,5 @@
         </collision>
       </link>
-      <link name="lidar_link">
+      <link name="base_laser">
         <inertial>
           <mass value="0.1"/>
@@ -131,5 +131,5 @@
         <origin xyz="0 0 0.5" rpy="0 0 0" />
         <parent link="base_link" />
-        <child link="lidar_link" />
+        <child link="base_laser" />
       </joint>
       <joint name="left_wheel_joint" type="continuous">
