Commit message: Fixed lidar location.
Rays can now be seen in gazebo, but the objects in the gazebo world
appear to be transparent to lidar

File: urdf/nubot.urdf.xacro (robot description, xacro)
@@ -31,5 +31,4 @@
       <link name="lidar_link">
         <inertial>
-        <origin xyz="0 0 0.5" rpy="0 0 0" />
           <mass value="0.1"/>
           <inertia
@@ -43,5 +42,4 @@
         </inertial>
         <collision>
-        <origin xyz="0 0 0.5" rpy="0 0 0" />
           <geometry>
             <box size="0.1 0.1 0.1" />
@@ -49,5 +47,4 @@
         </collision>
         <visual>
-        <origin xyz="0 0 0.5" rpy="0 0 0" />
           <geometry>
             <box size="0.1 0.1 0.1" />
@@ -132,4 +129,5 @@
       </link>
       <joint name="lidar_sensor_joint" type="fixed">
+        <origin xyz="0 0 0.5" rpy="0 0 0" />
         <parent link="chassis" />
         <child link="lidar_link" />

Commit message: Added base_footprint

File: urdf/nubot.urdf.xacro (robot description, xacro)
@@ -29,4 +29,10 @@
         </collision>
       </link>
+      <link name="base_footprint" />
+      <joint name="base_joint" type="fixed">
+             <parent link="base_link"/>
+             <child link="base_footprint"/>
+             <origin xyz="0.0 0.0 -0.15" rpy="0.0 0.0 0.0" />
+     </joint>
       <link name="base_laser">
         <inertial>
